Commit message: Updated visualization

File: src/micromouse_description/urdf/micromouse.urdf.xacro (robot description, xacro)
@@ -18,7 +18,7 @@
   <xacro:property name="ir_noise_stddev" value="0.005"/>
   <xacro:property name="ir_update_rate" value="20"/>
-  <material name="chassis_white"><color rgba="0.92 0.92 0.9 1"/></material>
-  <material name="wheel_black"><color rgba="0.1 0.1 0.1 1"/></material>
-  <material name="ir_dark"><color rgba="0.05 0.05 0.05 1"/></material>
+  <material name="chassis_blue"><color rgba="0.18 0.45 0.80 1"/></material>
+  <material name="wheel_dark"><color rgba="0.12 0.12 0.14 1"/></material>
+  <material name="sensor_red"><color rgba="0.85 0.15 0.15 1"/></material>
   <!-- ===================== base ===================== -->
   <link name="base_link">
@@ -26,5 +26,5 @@
       <origin xyz="0 0 ${base_z}" rpy="0 0 0"/>
       <geometry><box size="${base_size} ${base_size} ${base_height}"/></geometry>
-      <material name="chassis_white"/>
+      <material name="chassis_blue"/>
     </visual>
     <collision>
@@ -41,4 +41,12 @@
     </inertial>
   </link>
+  <!-- Low-friction chassis: a glancing touch of the chassis box against a
+       wall should SLIDE, not grip and spin the body off-axis (which slips the
+       wheels and races odometry ahead). Traction stays with the wheels
+       (mu=1.0); only the body shell is made slippery. -->
+  <gazebo reference="base_link">
+    <mu1>0.05</mu1>
+    <mu2>0.05</mu2>
+  </gazebo>
   <!-- ===================== wheels ===================== -->
   <xacro:macro name="wheel" params="prefix reflect">
@@ -47,5 +55,5 @@
         <origin xyz="0 0 0" rpy="1.5708 0 0"/>
         <geometry><cylinder radius="${wheel_radius}" length="${wheel_width}"/></geometry>
-        <material name="wheel_black"/>
+        <material name="wheel_dark"/>
       </visual>
       <collision>
@@ -79,5 +87,5 @@
       <visual>
         <geometry><sphere radius="${caster_radius}"/></geometry>
-        <material name="wheel_black"/>
+        <material name="wheel_dark"/>
       </visual>
       <collision>
@@ -109,5 +117,5 @@
       <visual>
         <geometry><box size="0.006 0.006 0.006"/></geometry>
-        <material name="ir_dark"/>
+        <material name="sensor_red"/>
       </visual>
       <inertial>
